Commit message: Moveit works, but in a different directory

File: urdf/george.urdf (robot description, URDF)
Before this commit: robot george, 101 links, 100 joints
Links:
- link base_link: geometry collision box size=.040 .02 .0365; visual mesh filename=package://george/meshes/torso_mm.dae scale=1 1 1
- link gripper_base: geometry collision box size=.005 .005 .005; visual mesh filename=package://george/meshes/gripper-base.dae scale=1 1 1
- link gripper_lfinger: geometry collision box size=.005 .005 .005; visual mesh filename=package://george/meshes/gripper-lfinger.dae scale=1 1 1
- link gripper_rfinger: geometry collision box size=.005 .005 .005; visual mesh filename=package://george/meshes/gripper-rfinger.dae scale=1 1 1
- link lfoot: geometry collision box size=0.065 0.002 0.15; visual mesh filename=package://george/meshes/foot.dae
- link lforearm1: geometry collision box size=.005 .005 .005; visual mesh filename=package://george/meshes/multi-purp-simple.dae scale=1 1 1
- link lforearm2: geometry collision box size=.005 .005 .005; visual mesh filename=package://george/meshes/multi-purp-simple.dae scale=1 1 1
- link lforearm3: geometry collision box size=.005 .005 .005; visual mesh filename=package://george/meshes/cbracket-simple.dae scale=1 1 1
- link lforearm4: geometry collision box size=.005 .005 .005; visual mesh filename=package://george/meshes/multi-purp-simple.dae scale=1 1 1
- link lforearm5: geometry collision box size=.005 .005 .005; visual mesh filename=package://george/meshes/lconnector-simple.dae scale=1 1 1
- link lknee1: geometry collision box size=.005 .005 .005; visual mesh filename=package://george/meshes/multi-purp-simple.dae scale=1 1 1
- link lknee2: geometry collision box size=.005 .005 .005; visual mesh filename=package://george/meshes/cbracket-simple.dae scale=1 1 1
- link lpleft: geometry collision box size=.005 .005 .005; visual mesh filename=package://george/meshes/low-profile-simple.dae scale=1 1 1
- link lpright: geometry collision box size=.005 .005 .005; visual mesh filename=package://george/meshes/low-profile-simple.dae scale=1 1 1
- link lshin1: geometry collision box size=.005 .005 .005; visual mesh filename=package://george/meshes/multi-purp-simple.dae scale=1 1 1
- link lshin2: geometry collision box size=.005 .005 .005; visual mesh filename=package://george/meshes/cbracket-simple.dae scale=1 1 1
- link lshin3: geometry collision box size=.005 .005 .005; visual mesh filename=package://george/meshes/multi-purp-simple.dae scale=1 1 1
- link lshoulder1: geometry collision box size=.005 .005 .005; visual mesh filename=package://george/meshes/offset-c-simple.dae scale=1 1 1
- link lthigh1: geometry collision box size=.005 .005 .005; visual mesh filename=package://george/meshes/cbracket-simple.dae scale=1 1 1
- link lthigh2: geometry collision box size=.005 .005 .005; visual mesh filename=package://george/meshes/multi-purp-simple.dae scale=1 1 1
- link lthigh3: geometry collision box size=.005 .005 .005; visual mesh filename=package://george/meshes/cbracket-simple.dae scale=1 1 1
- link lthigh4: geometry collision box size=.005 .005 .005; visual mesh filename=package://george/meshes/cbracket-simple.dae scale=1 1 1
- link rfoot: geometry collision box size=0.065 0.002 0.15; visual mesh filename=package://george/meshes/foot.dae
- link rforearm1: geometry collision box size=.005 .005 .005; visual mesh filename=package://george/meshes/multi-purp-simple.dae scale=1 1 1
- link rforearm2: geometry collision box size=.005 .005 .005; visual mesh filename=package://george/meshes/multi-purp-simple.dae scale=1 1 1
- link rknee1: geometry collision box size=.005 .005 .005; visual mesh filename=package://george/meshes/multi-purp-simple.dae scale=1 1 1
- link rknee2: geometry collision box size=.005 .005 .005; visual mesh filename=package://george/meshes/cbracket-simple.dae scale=1 1 1
- link rshin1: geometry collision box size=.005 .005 .005; visual mesh filename=package://george/meshes/multi-purp-simple.dae scale=1 1 1
- link rshin2: geometry collision box size=.005 .005 .005; visual mesh filename=package://george/meshes/cbracket-simple.dae scale=1 1 1
- link rshin3: geometry collision box size=.005 .005 .005; visual mesh filename=package://george/meshes/multi-purp-simple.dae scale=1 1 1
- link rshoulder1: geometry collision box size=.005 .005 .005; visual mesh filename=package://george/meshes/offset-c-simple.dae scale=1 1 1
- link rthigh1: geometry collision box size=.005 .005 .005; visual mesh filename=package://george/meshes/cbracket-simple.dae scale=1 1 1
- link rthigh2: geometry collision box size=.005 .005 .005; visual mesh filename=package://george/meshes/multi-purp-simple.dae scale=1 1 1
- link rthigh3: geometry collision box size=.005 .005 .005; visual mesh filename=package://george/meshes/cbracket-simple.dae scale=1 1 1
- link rthigh4: geometry collision box size=.005 .005 .005; visual mesh filename=package://george/meshes/cbracket-simple.dae scale=1 1 1

File: urdf/george.urdf.xacro (robot description, xacro)
@@ -10,5 +10,5 @@
     <visual>
       <geometry>
-	<mesh filename="package://george/meshes/torso_mm.dae" scale="0.0254 0.0254 0.0254"/>
+	<mesh filename="package://george/meshes/torso_mm.dae" scale="1 1 1"/>
       </geometry>
       <origin xyz="0 0 0" rpy="${M_PI/2} 0 ${M_PI}"/>
@@ -19,7 +19,7 @@
     <collision>
       <geometry>
-        <mesh filename="package://george/meshes/torso_mm.dae" scale="0.0254 0.0254 0.0254"/>
-      </geometry>
-      <origin xyz="0 0 0" rpy="${M_PI/2} 0 ${M_PI}"/>
+	      <box size=".040 .02 .0365"/>
+      </geometry>
+      <origin xyz="0 0 0" rpy="0 0 ${M_PI}"/>
     </collision>
 <!--       <inertial>
@@ -142,5 +142,5 @@
     <visual>
       <geometry>
-	<mesh filename="package://george/meshes/cbracket-simple.dae" scale="0.0254 0.0254 0.0254"/>
+	<mesh filename="package://george/meshes/cbracket-simple.dae" scale="1 1 1"/>
       </geometry>
       <origin xyz="${xyz}" rpy="${rpy}"/>
@@ -151,5 +151,6 @@
     <collision>
       <geometry>
-	<mesh filename="package://george/meshes/cbracket-simple.dae" scale="0.0254 0.0254 0.0254"/>
+        <box size=".005 .005 .005"/>
+	<!--  mesh filename="package://george/meshes/cbracket-simple.dae" scale="1 1 1"/-->
       </geometry>
       <origin xyz="${xyz}" rpy="${rpy}"/>
@@ -183,5 +184,5 @@
     <visual>
       <geometry>
-	<mesh filename="package://george/meshes/multi-purp-simple.dae" scale="0.0254 0.0254 0.0254"/>
+	<mesh filename="package://george/meshes/multi-purp-simple.dae" scale="1 1 1"/>
       </geometry>
       <origin xyz="${xyz}" rpy="${rpy}"/>
@@ -192,5 +193,6 @@
     <collision>
       <geometry>
-	<mesh filename="package://george/meshes/multi-purp-simple.dae" scale="0.0254 0.0254 0.0254"/>
+        <box size=".005 .005 .005"/>
+	<!--  mesh filename="package://george/meshes/multi-purp-simple.dae" scale="1 1 1"/-->
       </geometry>
       <origin xyz="${xyz}" rpy="${rpy}"/>
@@ -208,5 +210,5 @@
     <visual>
       <geometry>
-	<mesh filename="package://george/meshes/offset-c-simple.dae" scale="0.0254 0.0254 0.0254"/>
+	<mesh filename="package://george/meshes/offset-c-simple.dae" scale="1 1 1"/>
       </geometry>
       <origin xyz="0 0 0" rpy="${M_PI/2} 0 ${rot}"/>
@@ -217,5 +219,6 @@
     <collision>
       <geometry>
-	<mesh filename="package://george/meshes/offset-c-simple.dae" scale="0.0254 0.0254 0.0254"/>
+        <box size=".005 .005 .005"/>
+	<!-- mesh filename="package://george/meshes/offset-c-simple.dae" scale="1 1 1"/-->
       </geometry>
       <origin xyz="0 0 0" rpy="${M_PI/2} 0 ${rot}"/>
@@ -233,5 +236,5 @@
     <visual>
       <geometry>
-	<mesh filename="package://george/meshes/lconnector-simple.dae" scale="0.0254 0.0254 0.0254"/>
+	<mesh filename="package://george/meshes/lconnector-simple.dae" scale="1 1 1"/>
       </geometry>
       <origin xyz="0 0 0" rpy="0 0 ${rot}"/>
@@ -242,5 +245,6 @@
     <collision>
       <geometry>
-	<mesh filename="package://george/meshes/lconnector-simple.dae" scale="0.0254 0.0254 0.0254"/>
+        <box size=".005 .005 .005"/>
+	<!--  mesh filename="package://george/meshes/lconnector-simple.dae" scale="1 1 1"/-->
       </geometry>
       <origin xyz="0 0 0" rpy="0 0 ${rot}"/>
@@ -267,5 +271,5 @@
     <collision>
       <geometry>
-	<mesh filename="package://george/meshes/foot.dae"/>
+        <box size="0.065 0.002 0.15"/>
       </geometry>
       <origin xyz="0 0 0" rpy="0 0 0"/>
@@ -310,5 +314,5 @@
     <visual>
       <geometry>
-        <mesh filename="package://george/meshes/gripper-base.dae" scale="0.0254 0.0254 0.0254"/>
+        <mesh filename="package://george/meshes/gripper-base.dae" scale="1 1 1"/>
       </geometry>
       <origin xyz="0 0 0" rpy="0 ${-M_PI/2} 0"/>
@@ -317,4 +321,9 @@
       </material>
     </visual>
+    <collision>
+      <geometry>
+        <box size=".005 .005 .005"/>
+      </geometry>
+    </collision>
       <inertial>
         <mass value="0.001"/>
@@ -325,5 +334,5 @@
     <visual>
       <geometry>
-        <mesh filename="package://george/meshes/gripper-lfinger.dae" scale="0.0254 0.0254 0.0254"/>
+        <mesh filename="package://george/meshes/gripper-lfinger.dae" scale="1 1 1"/>
       </geometry>
       <origin xyz="0 0 0" rpy="0 0 0"/>
@@ -332,4 +341,9 @@
       </material>
     </visual>
+    <collision>
+      <geometry>
+        <box size=".005 .005 .005"/>
+      </geometry>
+    </collision>
       <inertial>
         <mass value="0.001"/>
@@ -347,5 +361,5 @@
     <visual>
       <geometry>
-        <mesh filename="package://george/meshes/gripper-rfinger.dae" scale="0.0254 0.0254 0.0254"/>
+        <mesh filename="package://george/meshes/gripper-rfinger.dae" scale="1 1 1"/>
       </geometry>
       <origin xyz="0 0 0" rpy="0 0 0"/>
@@ -354,4 +368,9 @@
       </material>
     </visual>
+    <collision>
+      <geometry>
+        <box size=".005 .005 .005"/>
+      </geometry>
+    </collision>
       <inertial>
         <mass value="0.001"/>
@@ -379,5 +398,5 @@
     <visual>
       <geometry>
-        <mesh filename="package://george/meshes/low-profile-simple.dae" scale="0.0254 0.0254 0.0254"/>
+        <mesh filename="package://george/meshes/low-profile-simple.dae" scale="1 1 1"/>
       </geometry>
       <origin xyz="0 0 0" rpy="-${M_PI/2} -${M_PI/2} 0"/>
@@ -388,5 +407,6 @@
     <collision>
       <geometry>
-        <mesh filename="package://george/meshes/low-profile-simple.dae" scale="0.0254 0.0254 0.0254"/>
+        <box size=".005 .005 .005"/>
+        <!--  mesh filename="package://george/meshes/low-profile-simple.dae" scale="1 1 1"/-->
       </geometry>
       <origin xyz="0 0 0" rpy="-${M_PI/2} -${M_PI/2} 0"/>
@@ -948,3 +968,75 @@
     </actuator>
   </transmission>
+  <transmission name="tran12">
+    <type>transmission_interface/SimpleTransmission</type>
+    <joint name="LShoulder"/>
+    <actuator name="motor12">
+      <hardwareInterface>EffortJointInterface</hardwareInterface>
+      <mechanicalReduction>1</mechanicalReduction>
+    </actuator>
+  </transmission>
+  <transmission name="tran13">
+    <type>transmission_interface/SimpleTransmission</type>
+    <joint name="LElbow"/>
+    <actuator name="motor13">
+      <hardwareInterface>EffortJointInterface</hardwareInterface>
+      <mechanicalReduction>1</mechanicalReduction>
+    </actuator>
+  </transmission>
+  <transmission name="tran14">
+    <type>transmission_interface/SimpleTransmission</type>
+    <joint name="LWristTwist" />
+    <actuator name="motor14">
+      <hardwareInterface>EffortJointInterface</hardwareInterface>
+      <mechanicalReduction>1</mechanicalReduction>
+    </actuator>
+  </transmission>
+  <transmission name="tran15">
+    <type>transmission_interface/SimpleTransmission</type>
+    <joint name="LWristFlex" />
+    <actuator name="motor15">
+      <hardwareInterface>EffortJointInterface</hardwareInterface>
+      <mechanicalReduction>1</mechanicalReduction>
+    </actuator>
+  </transmission>
+  <transmission name="tran16">
+    <type>transmission_interface/SimpleTransmission</type>
+    <joint name="RShoulder"/>
+    <actuator name="motor16">
+      <hardwareInterface>EffortJointInterface</hardwareInterface>
+      <mechanicalReduction>1</mechanicalReduction>
+    </actuator>
+  </transmission>
+  <transmission name="tran17">
+    <type>transmission_interface/SimpleTransmission</type>
+    <joint name="RElbow"/>
+    <actuator name="motor17">
+      <hardwareInterface>EffortJointInterface</hardwareInterface>
+      <mechanicalReduction>1</mechanicalReduction>
+    </actuator>
+  </transmission>
+  <transmission name="tran18">
+    <type>transmission_interface/SimpleTransmission</type>
+    <joint name="RWristTwist" />
+    <actuator name="motor18">
+      <hardwareInterface>EffortJointInterface</hardwareInterface>
+      <mechanicalReduction>1</mechanicalReduction>
+    </actuator>
+  </transmission>
+  <!--  transmission name="tran19">
+    <type>transmission_interface/SimpleTransmission</type>
+    <joint name="RHand" />
+    <actuator name="motor19">
+      <hardwareInterface>EffortJointInterface</hardwareInterface>
+      <mechanicalReduction>1</mechanicalReduction>
+    </actuator>
+  </transmission-->
+  <transmission name="tran20">
+    <type>transmission_interface/SimpleTransmission</type>
+    <joint name="Head" />
+    <actuator name="motor20">
+      <hardwareInterface>EffortJointInterface</hardwareInterface>
+      <mechanicalReduction>1</mechanicalReduction>
+    </actuator>
+  </transmission>
 </robot>

Commit message: Now working with simulation.

File: urdf/george.urdf (robot description, URDF)
Before this commit: robot george, 101 links, 100 joints
Links:
- added link torso_mass, mass 0.1; collision box size=.001 .001 .001; visual box size=.001 .001 .001
- link Head_servo_body: mass 0.045 -> 0.055
- link LAnkleBend_servo_body: mass 0.045 -> 0.055
- link LAnkleTilt_servo_body: mass 0.045 -> 0.055
- link LElbow_servo_body: mass 0.045 -> 0.055
- link LHip_servo_body: mass 0.045 -> 0.055
- link LKnee_servo_body: mass 0.045 -> 0.055
- link LShoulder_servo_body: mass 0.045 -> 0.055
- link LWaist_servo_body: mass 0.045 -> 0.055
- link LWristFlex_servo_body: mass 0.045 -> 0.055
- link LWristTwist_servo_body: mass 0.045 -> 0.055
- link RAnkleBend_servo_body: mass 0.045 -> 0.055
- link RAnkleTilt_servo_body: mass 0.045 -> 0.055
- link RElbow_servo_body: mass 0.045 -> 0.055
- link RHip_servo_body: mass 0.045 -> 0.055
- link RKnee_servo_body: mass 0.045 -> 0.055
- link RShoulder_servo_body: mass 0.045 -> 0.055
- link RWaist_servo_body: mass 0.045 -> 0.055
- link RWristTwist_servo_body: mass 0.045 -> 0.055
- link gripper_servo_body: mass 0.045 -> 0.055
- link lpleft_servo_servo_body: mass 0.045 -> 0.055
- link lpright_servo_servo_body: mass 0.045 -> 0.055
Joints:
- added joint torso_to_base: type fixed, parent base_link, child torso_mass, origin xyz=0 0 0 rpy=0 0 0

File: urdf/george.urdf.xacro (robot description, xacro)
@@ -7,4 +7,20 @@
 	<inertia ixx="0.001" ixy="0.0" ixz="0.0" iyy="0.001" iyz="0.0" izz="0.001"/>
   </xacro:macro>
+  <link name="torso_mass">
+      <visual>
+          <geometry>
+              <box size=".001 .001 .001"/>
+          </geometry>
+      </visual>
+      <collision>
+         <geometry>
+             <box size=".001 .001 .001"/>
+          </geometry>
+      </collision>
+      <inertial>
+          <inertia ixx="0.001" ixy="0.0" ixz="0.0" iyy="0.001" iyz="0.0" izz="0.001"/>
+          <mass value="0.4"/>
+      </inertial>
+  </link>
   <link name="base_link">
     <visual>
@@ -48,5 +64,5 @@
       </collision>
       <inertial>
-	<mass value="0.045"/>
+	<mass value="0.055"/>
 	<xacro:default_inertia/>
       </inertial>
@@ -435,4 +451,9 @@
   <!-- *********************************************************** -->
   <xacro:servo_bp prefix="LWaist" rot="${M_PI/2}" />
+  <joint name="torso_to_base" type="fixed">
+    <parent link="base_link"/>
+    <child link="torso_mass"/>
+    <origin xyz="0 0 0" rpy="0 0 0"/>
+  </joint>
   <joint name="torso_to_lwaist" type="fixed">
     <parent link="base_link"/>

Commit message: Now able to plan and move feet with python code.

File: urdf/george.urdf (robot description, URDF)
Before this commit: robot george, 102 links, 101 joints
Links:
- link torso_mass: mass 0.1 -> 0.4
Joints:
- joint gripper_lfinger_to_base: type prismatic -> fixed
- joint gripper_rfinger_to_base: type prismatic -> fixed

File: urdf/george.urdf.xacro (robot description, xacro)
@@ -122,5 +122,5 @@
       <origin xyz="0 0 0"/>
     </joint>
-  <joint name="${prefix}" type="revolute">
+  <joint name="${prefix}" type="revolute" >
     <axis xyz="0 0 -1"/>
     <limit effort="1000.0" lower="-${M_PI/2}" upper="${M_PI/2}" velocity="0.5"/>
@@ -367,5 +367,6 @@
       </inertial>
   </link>
-  <joint name="${name}_lfinger_to_base" type="prismatic">
+  <!--joint name="${name}_lfinger_to_base" type="prismatic"-->
+  <joint name="${name}_lfinger_to_base" type="fixed">
     <axis xyz="0 1 0"/>
     <parent link="${name}_base"/>
@@ -394,5 +395,6 @@
       </inertial>
   </link>
-  <joint name="${name}_rfinger_to_base" type="prismatic">
+  <joint name="${name}_rfinger_to_base" type="fixed">
+  <!--joint name="${name}_rfinger_to_base" type="prismatic"-->
     <axis xyz="0 1 0"/>
     <parent link="${name}_base"/>

Commit message: Fixed the gripper missing problem.

File: urdf/george.urdf (robot description, URDF)
Before this commit: robot george, 102 links, 101 joints
Links:
- removed link gripper_base
- removed link gripper_lfinger
- removed link gripper_rfinger
- removed link gripper_servo_body
- removed link gripper_servo_horn
- removed link gripper_servo_lip
- added link RHand_base, mass 0.001; collision box size=.005 .005 .005; visual mesh filename=package://george/meshes/gripper-base.dae scale=1 1 1
- added link RHand_lfinger, mass 0.001; collision box size=.005 .005 .005; visual mesh filename=package://george/meshes/gripper-lfinger.dae scale=1 1 1
- added link RHand_rfinger, mass 0.001; collision box size=.005 .005 .005; visual mesh filename=package://george/meshes/gripper-rfinger.dae scale=1 1 1
- added link RHand_servo_body, mass 0.055; collision box size=.040 .02 .0365; visual box size=.040 .02 .0365
- added link RHand_servo_horn, mass 0.001; collision cylinder length=0.001 radius=0.012; visual cylinder length=0.001 radius=0.012
- added link RHand_servo_lip, mass 0.001; collision box size=.0528 .02 .002; visual box size=.0528 .02 .002
Joints:
- removed joint gripper
- removed joint gripper_lfinger_to_base
- removed joint gripper_rfinger_to_base
- removed joint gripper_servo_lip_to_body
- removed joint gripper_servo_to_base
- added joint RHand_lfinger_to_base: type fixed, parent RHand_base, child RHand_lfinger, origin xyz=0 0 0 rpy=0 -1.5708 0, axis 0 1 0, limit lower=-0.005 upper=0.0137 effort=1000.0 velocity=0.5
- added joint RHand_rfinger_to_base: type fixed, parent RHand_base, child RHand_rfinger, origin xyz=0 0 0 rpy=0 -1.5708 0, axis 0 1 0, limit lower=-0.0137 upper=0.005 effort=1000.0 velocity=0.5
- added joint RHand_servo_lip_to_body: type fixed, parent RHand_servo_body, child RHand_servo_lip, origin xyz=0 0 0
- added joint RHand_servo_to_base: type fixed, parent RHand_base, child RHand_servo_body, origin xyz=0.0058 0.0095 0.01195 rpy=1.5708 0 -1.5708
- added joint rtip1: type fixed, parent RHand_base, child rtip1, origin xyz=0 0 0.070 rpy=0 1.5708 0, axis 0 0 1, limit lower=-1.5708 upper=1.5708 effort=1000.0 velocity=0.5
- joint RHand: axis 0 0 1 -> 0 0 -1; child rtip1 -> RHand_servo_horn; origin xyz=0 0 0.070 rpy=0 1.5708 0 -> xyz=.01 0 0.0161 rpy=0 0 0; parent gripper_base -> RHand_servo_body
- joint gripper_to_wrist: child gripper_base -> RHand_base

File: urdf/george.urdf.xacro (robot description, xacro)
@@ -818,8 +818,8 @@
     <origin xyz="${0.0134+.001} 0 -0.0142" rpy="${M_PI/2} 0 ${M_PI/2}"/>
   </joint>
-  <xacro:gripper name="gripper" />
+  <xacro:gripper name="RHand" />
   <joint name="gripper_to_wrist" type="fixed">
     <parent link="RWristTwist_servo_horn"/>
-    <child link="gripper_base"/>
+    <child link="RHand_base"/>
     <origin xyz="0 0 0" rpy="0 0 0"/>
   </joint>
@@ -835,8 +835,8 @@
     </visual>
   </link>
-  <joint name="RHand" type="revolute">
+  <joint name="rtip1" type="fixed">
     <axis xyz="0 0 1"/>
     <limit effort="1000.0" lower="-${M_PI/2}" upper="${M_PI/2}" velocity="0.5"/>
-    <parent link="gripper_base"/>
+    <parent link="RHand_base"/>
     <child link="rtip1"/>
     <origin xyz="0 0 0.070" rpy="0 ${M_PI/2} 0"/>
